File: digital_dice.kicad_sch (KiCad schematic)
At the start: 23 parts, among them J1 Barrel_Jack, SW1 SW_SPST, SW2 SW_SPST, U1 NE555D, U2 74LS90, U3 74LS47, U4 SC39-11EWA, U5 LM7805_TO220, U6 74LS11

Commit message: Final Touches:
Connections:
- net +5V: now reaches D1.1 (K), R10.1, SW1.1 (A), U1.8 (VCC), U2.2 (R0(1)), U2.3 (R0(2)), U2.5 (VCC), U3.16 (VCC), U3.3 (LT), U3.4 (BI), U3.5 (RBI), U6.14 (VCC)
- net DIS: now reaches R1.1, R10.2, U1.7 (DIS)
- net Q1: now reaches U2.9 (Q1), U3.1 (B), U6.2
- net Q2: now reaches U2.8 (Q2), U3.2 (C), U6.1
- net Q3: now reaches U2.11 (Q3), U3.6 (D)
- net Q0: now reaches U2.12 (Q0), U3.7 (A), U6.13
- net TR/THR: now reaches R1.2, U1.2 (TR), U1.6 (THR)
- net Q: now reaches U1.3 (Q), U2.1 (CP1..3)
Other:
- note added: "BCD DECODER (Binary → 7-Segment)"
- note added: "COUNTER (Random Number Generator)"
- note added: "DISPLAY OUTPUT"
- note added: "Github"
- note added: "SECTION 1: POWER SUPPLY (Input → Regulation)"
- note added: "SECTION 2: CLOCK GENERATOR (555 Timer Oscillator)"
- company: (none) -> Vladyslav Hirchuk - git: SoloScriptSage
- title: (none) -> Digital Dice
- moved on the sheet: C3, C4, C5, D1, J1, R1, R10, R2, R5, SW1, SW2, U1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
